File: PWR_PCB.kicad_pcb (KiCad board)
At the start: 2 copper layers, 70 x 70 mm, 56 parts, among them J1 BUZZER, J2 BURNER, J3 BATT, J4 BAKCBONE, Q1 PSMN7R0, Q2 PSMN7R0, U1 INA180A3, U2 BD9D320EFJ, U3 INA180A3, U4 BD9D320EFJ

Commit message: Added debug things
Parts:
- added J5: DEB, Connector_PinSocket_2.54mm:PinSocket_1x06_P2.54mm_Vertical, F.Cu at (92.5, 40.0)
- moved J1 9.50 mm to (134.5, 40.0)
- moved J2 9.50 mm to (123.5, 40.0)
- moved J3 9.50 mm to (114.8, 40.0)
- moved Q1 9.50 mm to (134.8, 45.7)
- moved Q2 9.50 mm to (123.6, 45.8)
- moved R10 9.50 mm to (126.5, 47.2)
- moved R9 9.50 mm to (137.5, 47.0)
Routing:
- net 3V3: track 43.3 -> 115.4 mm, vias 0 -> 3
- net 4V: track 20.4 -> 86.2 mm
- net BUZZER: track 73.6 -> 116.2 mm, vias 1 -> 2
- net BURNER: track 79.6 -> 106.9 mm, vias 1 -> 2
- net VDD: track 117.6 -> 127.2 mm
- net Net-(J2-Pad1): vias 0 -> 4
- net Net-(J1-Pad1): vias 0 -> 4
- net GND: vias 155 -> 205
- added copper zone on F.Cu, net 3V3
- added copper zone on F.Cu, net 4V
- added copper zone on B.Cu, net Net-(J1-Pad1)
- added copper zone on B.Cu, net Net-(J2-Pad1)
Other:
- board text added: "3V3"
- board text added: "4V"
- board text added: "BATT"
- board text added: "BURNER"
- board text added: "BUZZER"
- board text added: "CURR_3V3"
- board text added: "CURR_V4"
- board text added: "DEBUG"
- board text added: "GND"
- board text added: "VDD"
- board text added: "VOLT_SENSE"

Commit message: Reverse polarity protection
Parts:
- added Q3: SIA4371EDJ, Package_TO_SOT_SMD:Vishay_PowerPAK_SC70-6L_Single, F.Cu at (112.2, 43.4)
Connections:
- J3 pad 2: VDD -> /MISC/BATT
Routing:
- net VDD: track 127.2 -> 130.4 mm
- net GND: vias 205 -> 202
- added copper zone on F.Cu, net /MISC/BATT

Commit message: V1
Parts:
- J5: footprint Connector_PinSocket_2.54mm:PinSocket_1x06_P2.54mm_Vertical -> Connector_PinSocket_2.54mm:PinSocket_1x06_P2.54mm_Horizontal
- R1: value 22k -> 10k
- R11: value 55k -> 22k
- R12: value 55k -> 10k
- moved J5 13.8 mm to (105.3, 45.2), turned to -90 degrees
- moved C22 0.32 mm to (113.8, 67.1)
- moved C20 0.21 mm to (111.3, 73.1)
Connections:
- J5 pad 1: GND -> VDD
- J5 pad 2: 4V -> BURNER
- J5 pad 3: 3V3 -> BUZZER
- J5 pad 4: BUZZER -> 3V3
- J5 pad 5: BURNER -> 4V
- J5 pad 6: VDD -> GND
Routing:
- net VDD: track 130.4 -> 54.4 mm
- net 4V: track 86.2 -> 66.1 mm
- net 3V3: track 115.4 -> 97.5 mm
- net BUZZER: track 116.2 -> 110.8 mm
- net BURNER: track 106.9 -> 103.0 mm
- net GND: vias 202 -> 195
Other:
- board text added: "MADE BY BASEMENT PROJECT WASSUP PWR BOARD V1"
- board text removed: "DEBUG"
