File: PWR_PCB.kicad_sch (KiCad schematic)
At the start: 0 parts

Commit message: V1
Other:
- company: (none) -> BASEMENT
Changed lines of the file:
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@@
 (kicad_sch (version 20211123) (generator eeschema)
   (paper "A4")
+  (title_block
+    (date "%%date%%")
+    (rev "%%version%%")
+    (company "BASEMENT")
+  )
   (sheet (at 38.1 38.1) (size 25.4 25.4) (fields_autoplaced)
     (stroke (width 0.1524) (type solid) (color 0 0 0 0))
@@
   )
   (symbol_instances
+    (path "/9dc28bf4-24e4-44da-9bb5-0c98f1202cca/4483b82a-4c6d-49c7-ba50-4128496f2f68"
+      (reference "#FLG0101") (unit 1) (value "PWR_FLAG") (footprint "")
+    )
+    (path "/9dc28bf4-24e4-44da-9bb5-0c98f1202cca/4dd0a560-7dc2-4901-b564-77c087507c3f"
+      (reference "#FLG0102") (unit 1) (value "PWR_FLAG") (footprint "")
+    )
+    (path "/9dc28bf4-24e4-44da-9bb5-0c98f1202cca/3a4937a5-390f-4e22-8b17-9932d60db00d"
+      (reference "#FLG0103") (unit 1) (value "PWR_FLAG") (footprint "")
+    )
+    (path "/9dc28bf4-24e4-44da-9bb5-0c98f1202cca/b17facc3-47d6-4ff7-9b86-6381ccb0ad7b"
+      (reference "#FLG0104") (unit 1) (value "PWR_FLAG") (footprint "")
+    )
     (path "/08a162f4-e79c-43d8-b22f-cfc45b757ccd/4408e293-f6fa-4a92-b869-d3c74ead88ea"
       (reference "#PWR0101") (unit 1) (value "GND") (footprint "")
@@
     )
     (path "/9dc28bf4-24e4-44da-9bb5-0c98f1202cca/bd82afa9-9709-4a9b-881a-0afd8f2d020e"
-      (reference "#PWR?") (unit 1) (value "GND") (footprint "")
+      (reference "#PWR0136") (unit 1) (value "GND") (footprint "")
     )
     (path "/08a162f4-e79c-43d8-b22f-cfc45b757ccd/dfc9e2eb-6f2d-4605-a917-9b5e2c5c87b1"
@@
     )
     (path "/9dc28bf4-24e4-44da-9bb5-0c98f1202cca/76a38dab-7841-4eb3-9aac-e54a29452de0"
-      (reference "J5") (unit 1) (value "DEB") (footprint "Connector_PinSocket_2.54mm:PinSocket_1x06_P2.54mm_Vertical")
+      (reference "J5") (unit 1) (value "DEB") (footprint "Connector_PinSocket_2.54mm:PinSocket_1x06_P2.54mm_Horizontal")
     )
     (path "/08a162f4-e79c-43d8-b22f-cfc45b757ccd/0dc88c26-cabf-41f4-9e46-4f028253120e"
