File: power3v3.kicad_sch (KiCad schematic)
At the start: 21 parts, among them U3 INA180A3, U4 BD9D320EFJ

Commit message: First version for PCB
Parts:
- R5, R6, R7: footprint Resistor_SMD:R_0603_1608Metric -> Resistor_SMD:R_0402_1005Metric
Changed lines of the file:
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@@
       (effects (font (size 1.27 1.27)) (justify right))
     )
-    (property "Footprint" "Resistor_SMD:R_0603_1608Metric" (id 2) (at 124.46 73.66 0)
+    (property "Footprint" "Resistor_SMD:R_0402_1005Metric" (id 2) (at 124.46 73.66 0)
       (effects (font (size 1.27 1.27)) hide)
     )
@@
       (effects (font (size 1.27 1.27)) (justify right))
     )
-    (property "Footprint" "Resistor_SMD:R_0603_1608Metric" (id 2) (at 124.46 66.04 0)
+    (property "Footprint" "Resistor_SMD:R_0402_1005Metric" (id 2) (at 124.46 66.04 0)
       (effects (font (size 1.27 1.27)) hide)
     )
@@
       (effects (font (size 1.27 1.27)) (justify right))
     )
-    (property "Footprint" "Resistor_SMD:R_0603_1608Metric" (id 2) (at 80.01 60.96 0)
-      (effects (font (size 1.27 1.27)) hide)
-    )
+    (property "Footprint" "Resistor_SMD:R_0402_1005Metric" (id 2) (at 80.01 60.96 0)
+      (effects (font (size 1.27 1.27)) hide)
+    )

Commit message: V1
Other:
- company: (none) -> BASEMENT
Changed lines of the file:
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@@
 (kicad_sch (version 20211123) (generator eeschema)
   (paper "A4")
+  (title_block
+    (date "%%date%%")
+    (rev "%%version%%")
+    (company "BASEMENT")
+  )
   (junction (at 39.37 39.37) (diameter 0) (color 0 0 0 0)
   )
