File: power4v.kicad_sch (KiCad schematic)
At the start: 23 parts, among them U1 INA180A3, U2 BD9D320EFJ

Commit message: First version for PCB
Parts:
- R1, R2, R3: footprint Resistor_SMD:R_0603_1608Metric -> Resistor_SMD:R_0402_1005Metric
- R4: footprint Resistor_SMD:R_0603_1608Metric -> LOCAL:0508
Changed lines of the file:
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@@
       (effects (font (size 1.27 1.27)) (justify right))
     )
-    (property "Footprint" "Resistor_SMD:R_0603_1608Metric" (id 2) (at 76.2 57.15 0)
+    (property "Footprint" "Resistor_SMD:R_0402_1005Metric" (id 2) (at 76.2 57.15 0)
       (effects (font (size 1.27 1.27)) hide)
     )
@@
       (effects (font (size 1.27 1.27)) (justify right))
     )
-    (property "Footprint" "Resistor_SMD:R_0603_1608Metric" (id 2) (at 120.65 62.23 0)
+    (property "Footprint" "Resistor_SMD:R_0402_1005Metric" (id 2) (at 120.65 62.23 0)
       (effects (font (size 1.27 1.27)) hide)
     )
@@
       (effects (font (size 1.27 1.27)) (justify right))
     )
-    (property "Footprint" "Resistor_SMD:R_0603_1608Metric" (id 2) (at 212.09 52.07 0)
+    (property "Footprint" "LOCAL:0508" (id 2) (at 212.09 52.07 0)
       (effects (font (size 1.27 1.27)) hide)
     )
@@
       (effects (font (size 1.27 1.27)) (justify right))
     )
-    (property "Footprint" "Resistor_SMD:R_0603_1608Metric" (id 2) (at 120.65 69.85 0)
-      (effects (font (size 1.27 1.27)) hide)
-    )
+    (property "Footprint" "Resistor_SMD:R_0402_1005Metric" (id 2) (at 120.65 69.85 0)
+      (effects (font (size 1.27 1.27)) hide)
+    )

Commit message: Changed ressistor values
Parts:
- R1: value 22k -> 10k
Changed lines of the file:
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@@
       (effects (font (size 1.27 1.27)) (justify right))
     )
-    (property "Value" "22k" (id 1) (at 73.66 58.4199 0)
+    (property "Value" "10k" (id 1) (at 73.66 58.4199 0)
       (effects (font (size 1.27 1.27)) (justify right))
     )

Commit message: V1
Other:
- company: (none) -> BASEMENT
Changed lines of the file:
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@@
 (kicad_sch (version 20211123) (generator eeschema)
   (paper "A4")
+  (title_block
+    (date "%%date%%")
+    (rev "%%version%%")
+    (company "BASEMENT")
+  )
   (junction (at 31.75 43.18) (diameter 0) (color 0 0 0 0)
   )
